Commit message: add controller module

File: model/braccio_arm.urdf (robot description, URDF)
Before this commit: robot braccio, 9 links, 8 joints
Joints:
- joint base_joint: limit lower=0.0 upper=3.1416 effort=1.0 velocity=1.0 -> lower=0.0 upper=3.1416 effort=1000.0 velocity=1.0
- joint elbow_joint: limit lower=0 upper=3.1416 effort=1.0 velocity=1.0 -> lower=0 upper=3.1416 effort=1000.0 velocity=1.0
- joint gripper_joint: limit lower=0.1750 upper=1.2741 effort=1.0 velocity=1.0 -> lower=0.1750 upper=1.2741 effort=1000.0 velocity=1.0
- joint shoulder_joint: limit lower=0.2618 upper=2.8798 effort=1.0 velocity=1.0 -> lower=0.2618 upper=2.8798 effort=1000.0 velocity=1.0
- joint sub_gripper_joint: limit lower=1.2741 upper=2.3732 effort=1.0 velocity=1.0 -> lower=1.2741 upper=2.3732 effort=1000.0 velocity=1.0
- joint wrist_pitch_joint: limit lower=0 upper=3.1416 effort=1.0 velocity=1.0 -> lower=0 upper=3.1416 effort=1000.0 velocity=1.0
- joint wrist_roll_joint: limit lower=0.0 upper=3.1416 effort=1.0 velocity=1.0 -> lower=0.0 upper=3.1416 effort=1000.0 velocity=1.0
