Commit message: pybullet tryout

File: model/braccio_arm_clean.urdf (robot description, URDF)
Before this commit: robot braccio, 9 links, 8 joints
Links:
- removed link braccio_base_link
- removed link elbow_link
- removed link shoulder_link
- removed link world
- removed link wrist_pitch_link
- removed link wrist_roll_link
- added link link_1, mass 0.1; collision mesh filename=./braccio_arm_stl/braccio_base.stl scale=0.001 0.001 0.001; visual mesh filename=./braccio_arm_stl/braccio_base.stl scale=0.001 0.001 0.001
- added link link_2, mass 0.1; collision mesh filename=./braccio_arm_stl/braccio_shoulder.stl scale=0.001 0.001 0.001; visual mesh filename=./braccio_arm_stl/braccio_shoulder.stl scale=0.001 0.001 0.001
- added link link_3, mass 0.1; collision mesh filename=./braccio_arm_stl/braccio_elbow.stl scale=0.001 0.001 0.001; visual mesh filename=./braccio_arm_stl/braccio_elbow.stl scale=0.001 0.001 0.001
- added link link_4, mass 0.1; collision mesh filename=./braccio_arm_stl/braccio_wrist_pitch.stl scale=0.001 0.001 0.001; visual mesh filename=./braccio_arm_stl/braccio_wrist_pitch.stl scale=0.001 0.001 0.001
- added link link_5, mass 0.1; collision mesh filename=./braccio_arm_stl/braccio_wrist_roll.stl scale=0.001 0.001 0.001; visual mesh filename=./braccio_arm_stl/braccio_wrist_roll.stl scale=0.001 0.001 0.001
- link base_link: mass 2 -> 0.1
- link left_gripper_link: geometry collision mesh filename=./braccio_arm_stl/braccio_left_gripper.stl scale=0.001 0.001 0.001; visual mesh filename=./braccio_arm_stl/braccio_left_gripper.stl scale=0.001 0.001 0.001
- link right_gripper_link: geometry collision mesh filename=./braccio_arm_stl/braccio_right_gripper.stl scale=0.001 0.001 0.001; visual mesh filename=./braccio_arm_stl/braccio_right_gripper.stl scale=0.001 0.001 0.001
Joints:
- removed joint world_joint
- joint base_joint: child braccio_base_link -> link_1
- joint elbow_joint: child elbow_link -> link_3; parent shoulder_link -> link_2
- joint gripper_joint: limit lower=0.1750 upper=1.2741 effort=1000.0 velocity=1.0 -> lower=0.1750 upper=1.2741 effort=10.0 velocity=1.0; parent wrist_roll_link -> link_5
- joint shoulder_joint: child shoulder_link -> link_2; parent braccio_base_link -> link_1
- joint sub_gripper_joint: limit lower=1.2741 upper=2.3732 effort=1000.0 velocity=1.0 -> lower=0.1750 upper=1.2741 effort=10.0 velocity=1.0; mimic joint=gripper_joint -> (none); parent wrist_roll_link -> link_5
- joint wrist_pitch_joint: child wrist_pitch_link -> link_4; parent elbow_link -> link_3
- joint wrist_roll_joint: child wrist_roll_link -> link_5; parent wrist_pitch_link -> link_4

Commit message: gym environment ready

File: model/braccio_arm_clean.urdf (robot description, URDF)
Before this commit: robot braccio_arm, 8 links, 7 joints
Links:
- added link world
Joints:
- added joint world_joint: type fixed, parent world, child base_link, origin xyz=0.0 0.0 0.0 rpy=0.0 0.0 0.0
